Commit message: Phase 3: floating base, hydrodynamics, disturbances, base sensing
- MJCF: auv_base becomes a MuJoCo <freejoint/> in a fluid medium (ellipsoid
  fluid model => drag + added mass). Neutral buoyancy modelled as zero gravity
  (MuJoCo has no Archimedes buoyancy); documented Fossen upgrade path. Cube
  grown to 0.6 m to match the URDF.
- MujocoSystem: exposes the floating base as a 13-interface ros2_control sensor
  (auv_base pose+twist), subscribes /riptide/disturbance and applies wrenches to
  xfrc_applied, echoes /riptide/disturbance/ground_truth, and broadcasts
  world->auv_base_link TF + /riptide/odom via an internal spun node. Step count
  per write() is clamped so scheduling gaps cannot fast-forward the physics.
- URDF: world->base joint is now "floating" (RSP no longer publishes it; TF
  comes from the sim); base sensor declared in the ros2_control block.
- riptide_disturbance: new scenario generator node (none/steady_current/
  sinusoid/impulse), publishing DisturbanceCommand.
- Launch: disturbance arg + generator, mock-path static base TF.
- .gitignore: drop the accidentally-tracked .claude local/temp settings.

Verified: vehicle hovers at rest, a current drives it to a drag-limited speed,
the base drifts/oscillates under disturbance, base sensor + TF + odom + ground
truth all publish. EE-stabilization-under-disturbance needs the Phase 4
task-space controller.

Co-Authored-By: Claude Opus 4.8 <noreply@anthropic.com>

File: riptide_description/urdf/auv_base.xacro (robot description, xacro)
@@ -3,19 +3,18 @@
   <!--
     AUV base: a plain cube stand-in for the hull (per request).
-    Phase 1 attaches the cube to `world` with a FIXED joint so the arm loop can
-    be brought up against mock hardware. Phase 3 removes that fixed joint and
-    replaces it with a MuJoCo free joint + a floating-base state "sensor"
-    (base pose/twist exposed as ros2_control state interfaces) — the arm and
-    ros2_control blocks do not change.
+    Phase 3: the base is FLOATING. The world->base joint is of type "floating",
+    so robot_state_publisher does not publish that transform — instead the
+    MuJoCo SystemInterface broadcasts world->${name}_link TF from the simulated
+    free-joint pose (and exposes base pose/twist as a ros2_control sensor).
+    `${name}_link` is therefore the cube center (the frame MuJoCo publishes).
     A dedicated `${name}_mount_link` on the top face gives the arm a clean,
-    unambiguous mounting frame (the vendor bravo_7 joint carries a redundant
-    <origin>, so we never rely on its mount offset).
+    unambiguous mounting frame.
   -->
   <xacro:macro name="auv_base" params="parent name size mass">
-    <!-- Lift the cube so it rests with its bottom face on the world origin. -->
-    <joint name="${name}_joint" type="fixed">
+    <!-- Floating base: transform supplied at runtime (TF), not by RSP. -->
+    <joint name="${name}_joint" type="floating">
       <parent link="${parent}"/>
       <child link="${name}_link"/>
-      <origin xyz="0 0 ${size / 2.0}" rpy="0 0 0"/>
+      <origin xyz="0 0 0" rpy="0 0 0"/>
     </joint>
     <link name="${name}_link">

File: riptide_description/urdf/riptide.ros2_control.xacro (robot description, xacro)
@@ -31,4 +31,22 @@
     </joint>
   </xacro:macro>
+  <!-- Floating-base pose + twist, exposed as a ros2_control sensor (Phase 3). -->
+  <xacro:macro name="riptide_base_sensor" params="name">
+    <sensor name="${name}">
+      <state_interface name="position.x"/>
+      <state_interface name="position.y"/>
+      <state_interface name="position.z"/>
+      <state_interface name="orientation.x"/>
+      <state_interface name="orientation.y"/>
+      <state_interface name="orientation.z"/>
+      <state_interface name="orientation.w"/>
+      <state_interface name="linear_velocity.x"/>
+      <state_interface name="linear_velocity.y"/>
+      <state_interface name="linear_velocity.z"/>
+      <state_interface name="angular_velocity.x"/>
+      <state_interface name="angular_velocity.y"/>
+      <state_interface name="angular_velocity.z"/>
+    </sensor>
+  </xacro:macro>
   <xacro:macro name="riptide_ros2_control" params="name arm_prefix use_mock_hardware">
     <ros2_control name="${name}" type="system">
@@ -38,7 +56,8 @@
         </xacro:if>
         <xacro:unless value="${use_mock_hardware}">
-          <!-- Phase 2: identical joint interfaces below, real dynamics behind. -->
           <plugin>riptide_mujoco/MujocoSystem</plugin>
           <param name="mjcf_model">$(find riptide_description)/mujoco/riptide.xml</param>
+          <param name="floating_base_joint">auv_freejoint</param>
+          <param name="base_link_frame">auv_base_link</param>
         </xacro:unless>
       </hardware>
@@ -51,4 +70,6 @@
       <xacro:riptide_arm_joint jname="${arm_prefix}_joint6"/>
       <xacro:riptide_arm_joint jname="${arm_prefix}_joint7"/>
+      <!-- Floating-base sensor (MuJoCo populates it; mock reports zeros). -->
+      <xacro:riptide_base_sensor name="auv_base"/>
     </ros2_control>
   </xacro:macro>

File: riptide_description/urdf/riptide.urdf.xacro (robot description, xacro)
@@ -15,6 +15,6 @@
   <!-- World anchor. Phase 3 replaces this fixed attachment with a free joint. -->
   <link name="world"/>
-  <!-- Cube hull: 0.5 m, 80 kg (roughly a small work-class AUV footprint). -->
-  <xacro:auv_base parent="world" name="auv_base" size="0.5" mass="80.0"/>
+  <!-- Cube hull: 0.6 m, 80 kg (matches the MuJoCo scene). -->
+  <xacro:auv_base parent="world" name="auv_base" size="0.6" mass="80.0"/>
   <!-- Franka fer mounted on the center of the cube's top face. -->
   <xacro:franka_fer parent="auv_base_mount_link" robot_type="$(arg arm_type)">
