Commit message: Phase 4b: hull thrusters + base dynamic-positioning controller
Add 5 hull thrusters and a controller that station-keeps the AUV base so the
arm no longer fights an unbounded base drift.

Simulation (generate_scene.py -> riptide.xml):
- 5 force actuators on the base: 1 surge (+/-x) and 4 vertical corner
  thrusters (+/-z). Common mode = heave; left/right diff = roll; front/back
  diff = pitch. Each is a MuJoCo <motor> applied at a body-fixed site.

Seam (riptide.ros2_control.xacro + MujocoSystem):
- Expose the thrusters as a ros2_control <gpio>, one force command + applied-
  force state interface each, mapped by name to the MuJoCo actuators. Same
  declarative "add-an-actuator" pattern as the arm joints; GenericSystem
  handles it on the mock path too.

Controller (BaseThrusterController, runs alongside the EE controller):
- Reads the base sensor, computes a PD wrench [Fx, Fz, Mx, My] (surge/heave
  position hold + roll/pitch leveling), and allocates it to per-thruster
  forces via the pseudo-inverse of an allocation matrix rebuilt from the
  thruster geometry (positions + axes in config). Captures its hold pose on
  the first finite cycle and clamps to the thruster force limit.

Launch: new base_control arg (default true) spawns it; set false to A/B the
free-floating base.

Verified under a sinusoidal surge current: surge x held within a few cm,
heave z held exactly, roll/pitch level (qx,qy ~ 0), vs. the base drifting
past 1 m without it. Sway (y) and yaw are intentionally unactuated.

File: riptide_description/urdf/riptide.ros2_control.xacro (robot description, xacro)
@@ -30,4 +30,12 @@
       </state_interface>
     </joint>
+  </xacro:macro>
+  <!-- Hull thrusters (Phase 4b), exposed as a ros2_control gpio. Each thruster
+       is a force-commanded actuator mapped by name to a MuJoCo <motor>; the
+       matching state interface reports the applied force. Adding/removing a
+       thruster is a declarative change here + one entry in generate_scene.py. -->
+  <xacro:macro name="riptide_thruster" params="tname">
+    <command_interface name="${tname}"/>
+    <state_interface name="${tname}"/>
   </xacro:macro>
   <!-- Floating-base pose + twist, exposed as a ros2_control sensor (Phase 3). -->
@@ -72,4 +80,13 @@
       <!-- Floating-base sensor (MuJoCo populates it; mock reports zeros). -->
       <xacro:riptide_base_sensor name="auv_base"/>
+      <!-- Hull thruster bank (Phase 4b base dynamic positioning). Names match
+           the MuJoCo thruster actuators in generate_scene.py. -->
+      <gpio name="thrusters">
+        <xacro:riptide_thruster tname="thr_surge"/>
+        <xacro:riptide_thruster tname="thr_vfl"/>
+        <xacro:riptide_thruster tname="thr_vfr"/>
+        <xacro:riptide_thruster tname="thr_vbl"/>
+        <xacro:riptide_thruster tname="thr_vbr"/>
+      </gpio>
     </ros2_control>
   </xacro:macro>

Commit message: feat: switch for water,floating dynamics and wind currents

File: riptide_description/urdf/riptide.ros2_control.xacro (robot description, xacro)
@@ -57,5 +57,6 @@
     </sensor>
   </xacro:macro>
-  <xacro:macro name="riptide_ros2_control" params="name arm_prefix use_mock_hardware">
+  <xacro:macro name="riptide_ros2_control"
+               params="name arm_prefix use_mock_hardware water:=^|true fixed_base:=^|false">
     <ros2_control name="${name}" type="system">
       <hardware>
@@ -68,4 +69,7 @@
           <param name="floating_base_joint">auv_freejoint</param>
           <param name="base_link_frame">auv_base_link</param>
+          <!-- Reusability toggles (see MujocoSystem::on_init). -->
+          <param name="water">${water}</param>
+          <param name="fixed_base">${fixed_base}</param>
         </xacro:unless>
       </hardware>

File: riptide_description/urdf/riptide.urdf.xacro (robot description, xacro)
@@ -9,4 +9,9 @@
   <!-- Franka model + joint-name prefix (fer_joint1..7). -->
   <xacro:arg name="arm_type" default="fer"/>
+  <!-- Reusability toggles (MuJoCo path only):
+         water      -> fluid medium on/off (drag, added mass, current)
+         fixed_base -> weld the base to the world (non-floating manipulator) -->
+  <xacro:arg name="water" default="true"/>
+  <xacro:arg name="fixed_base" default="false"/>
   <xacro:include filename="$(find riptide_description)/urdf/common.xacro"/>
   <xacro:include filename="$(find riptide_description)/urdf/auv_base.xacro"/>
@@ -25,4 +30,6 @@
     name="RiptideSystem"
     arm_prefix="$(arg arm_type)"
-    use_mock_hardware="$(arg use_mock_hardware)"/>
+    use_mock_hardware="$(arg use_mock_hardware)"
+    water="$(arg water)"
+    fixed_base="$(arg fixed_base)"/>
 </robot>
