Commit message: feat: EE pose teleop GUI, inspection pipe, parallel MuJoCo viewer, build helper
- riptide_control: EeStabilizationController tracks a live desired pose on
  /riptide/ee_target (geometry_msgs/PoseStamped, world frame) and echoes the
  current target (latched) on /riptide/ee_target/current so teleop can seed
  itself without snapping the arm.
- riptide_bringup:
  * ee_target_gui.py - Tkinter teleop, press-and-hold arrows for XYZ + RPY
    (ee_gui:=true); ROS logic split from the Tk view and unit-tested.
  * mujoco_viewer.py - passive MuJoCo viewer mirroring the sim in parallel
    with RViz (mujoco_viewer:=true); spins ROS in a background thread and
    prefers X11 only when the GLFW build supports it.
  * reaper matches script filenames (mujoco_viewer.py / ee_target_gui.py) so
    it never kills the launch itself via its own args.
- riptide_description: add a subsea inspection pipe (r=0.5 m, 25 m) as a
  collidable geom in the MJCF and a matching static link in the URDF - shown in
  both viewers and within the arm's reach.
- build.sh: one-step ROS source + colcon build + overlay source (source it).
- README documents the new args/scenarios; .gitignore MUJOCO_LOG.TXT.

Co-Authored-By: Claude Opus 4.8 <noreply@anthropic.com>

File: riptide_description/urdf/riptide.urdf.xacro (robot description, xacro)
@@ -22,4 +22,30 @@
   <!-- Cube hull: 0.6 m, 80 kg (matches the MuJoCo scene). -->
   <xacro:auv_base parent="world" name="auv_base" size="0.6" mass="80.0"/>
+  <!-- Inspection target: a subsea pipe (solid cylinder, r=0.5 m, 25 m long),
+       static in the world. Mirrors the 'pipe' geom in mujoco/generate_scene.py
+       so RViz and the MuJoCo viewer agree. URDF cylinders lie along Z, so the
+       visual/collision are rolled +90 deg about X to lie along world Y. -->
+  <link name="pipe">
+    <visual>
+      <origin xyz="0 0 0" rpy="1.5707963 0 0"/>
+      <geometry>
+        <cylinder radius="0.5" length="25.0"/>
+      </geometry>
+      <material name="pipe_grey">
+        <color rgba="0.55 0.55 0.60 1"/>
+      </material>
+    </visual>
+    <collision>
+      <origin xyz="0 0 0" rpy="1.5707963 0 0"/>
+      <geometry>
+        <cylinder radius="0.5" length="25.0"/>
+      </geometry>
+    </collision>
+  </link>
+  <joint name="pipe_joint" type="fixed">
+    <parent link="world"/>
+    <child link="pipe"/>
+    <origin xyz="1.0 0 1.0" rpy="0 0 0"/>
+  </joint>
   <!-- Franka fer mounted on the center of the cube's top face. -->
   <xacro:franka_fer parent="auv_base_mount_link" robot_type="$(arg arm_type)">
